File: Hardware/Boards/FullBoard/FullBoard.kicad_pcb (KiCad board)
At the start: 2 copper layers, 19 parts, among them J1 Conn_01x03_Pin, J2 Conn_01x03_Pin, J3 Conn_01x03_Pin, J4 Conn_01x03_Pin, K1 Relay_SPDT, K2 Relay_SPDT, K3 Relay_SPDT, U1 GY-8511 UV sensor, U2 TEMT6000, U4 DS18B20-air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

Commit message: The full board combined
Parts:
- removed K2, K3: Relay_SPDT, Diplomna:Relay
- removed LA1, LA2: Lamp, Diplomna:Lamp
- removed R3: Heater, Diplomna:Heater
- added REF**: MountingHole_2.5mm_Pad_TopBottom, MountingHole:MountingHole_2.5mm_Pad_TopBottom, F.Cu at (156.7, 63.8)
- added REF**: MountingHole_2.5mm_Pad_TopBottom, MountingHole:MountingHole_2.5mm_Pad_TopBottom, F.Cu at (191.8, 63.8)
- added REF**: MountingHole_2.5mm_Pad_TopBottom, MountingHole:MountingHole_2.5mm_Pad_TopBottom, F.Cu at (191.8, 88.6)
- added REF**: MountingHole_2.5mm_Pad_TopBottom, MountingHole:MountingHole_2.5mm_Pad_TopBottom, F.Cu at (156.7, 88.6)
- moved K1 102.5 mm to (254.5, 101.1), turned to -90 degrees
- moved U2 97.6 mm to (75.7, 94.0)
- moved U1 96.3 mm to (68.1, 97.2)
- moved R1 92.5 mm to (63.8, 74.2), turned to 180 degrees
- moved U4 81.0 mm to (65.5, 87.4)
- moved J3 73.1 mm to (72.6, 62.5), turned to -90 degrees
- moved J4 72.6 mm to (72.6, 80.4), turned to -90 degrees
- moved J2 48.6 mm to (100.6, 80.4), turned to 90 degrees
- moved J1 45.9 mm to (100.6, 62.5), turned to 90 degrees
- moved U7 45.9 mm to (177.0, 105.4)
- moved U6 18.6 mm to (151.2, 70.3), turned to 90 degrees
- moved U5 17.1 mm to (160.3, 105.9)
- moved R2 5.09 mm to (159.0, 97.8), turned to 180 degrees
- moved U3 4.47 mm to (126.0, 76.7), turned to 180 degrees
Routing:
- net +3.3V: track 0.00 -> 166.3 mm
- net /Water level Power: track 0.00 -> 143.7 mm, vias 0 -> 1
- net GND: track 0.00 -> 139.9 mm, vias 0 -> 1
- net /WaterTemp: track 0.00 -> 132.7 mm, vias 0 -> 2
- net /Temp_Air: track 0.00 -> 110.9 mm, vias 0 -> 2
- net /Brightness: track 0.00 -> 110.4 mm, vias 0 -> 2
- net /UV: track 0.00 -> 105.5 mm, vias 0 -> 2
- net /Water level: track 0.00 -> 78.3 mm
- net +3V3: track 0.00 -> 65.7 mm
- net GND1: track 0.00 -> 61.7 mm
- net /UV_ref_main: track 0.00 -> 61.0 mm
- net /Air Temp: track 0.00 -> 30.9 mm
- net /Turbidity: track 0.00 -> 16.7 mm
- net /UV_OUT: track 0.00 -> 16.1 mm
- net /BRIGHTNESS_OUT: track 0.00 -> 13.0 mm
Other:
- board outline added: 153.9 x 70.1 mm
