File: Hardware/Boards/FullBoard/FullBoard.kicad_pcb (KiCad board)
At the start: 2 copper layers, 153.9 x 70.1 mm, 18 parts, among them J1 Conn_01x03_Pin, J2 Conn_01x03_Pin, J3 Conn_01x03_Pin, J4 Conn_01x03_Pin, K1 Relay_SPDT, U1 GY-8511 UV sensor, U2 TEMT6000, U4 DS18B20-air, U5 DS18B20-water, U6 Turbidity sensor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

Commit message: Almost completed scheme
Parts:
- added J5: Relay_Input, Diplomna:6pin_holes, F.Cu at (193.7, 48.9)
- moved U2 10.2 mm to (85.9, 93.9)
- moved R1 10.2 mm to (73.9, 74.0)
- moved J3 10.2 mm to (82.8, 62.4)
- moved J4 10.2 mm to (82.8, 80.2)
- moved U1 10.2 mm to (78.2, 97.0)
- moved U4 10.2 mm to (75.7, 87.2)
Connections:
- J4 pad 1: /Air Temp -> (no net)
- J4 pad 2: /BRIGHTNESS_OUT -> (no net)
- J4 pad 3: /UV_OUT -> (no net)
- R1 pad 2: /Air Temp -> (no net)
- U1 pad 4: /UV_OUT -> (no net)
- U2 pad 1: /BRIGHTNESS_OUT -> (no net)
- U4 pad 2: /Air Temp -> (no net)
Routing:
- net (no net): track 0.00 -> 58.4 mm
- net /Air Temp: track 30.9 -> 0.00 mm
- net /UV_OUT: track 16.1 -> 0.00 mm
- net /BRIGHTNESS_OUT: track 13.0 -> 0.00 mm
- net GND1: track 61.7 -> 53.2 mm
- net /Water level Power: track 143.7 -> 136.5 mm
- net /Temp_Air: track 110.9 -> 106.5 mm
- net /Turbidity: track 16.7 -> 13.6 mm
- net /UV: track 105.5 -> 103.5 mm
- net /Brightness: track 110.4 -> 108.9 mm
- net /WaterTemp: track 132.7 -> 131.8 mm
- removed copper zone on F.Cu, net GND
Other:
- board size 153.9 x 70.1 mm -> 138 x 70.1 mm
