File: Hardware/Boards/V2 - 1 board/FullBoard/FullBoard.kicad_sch (KiCad schematic)
At the start: 16 parts, among them J2 Conn_01x03_Pin, J3 Conn_01x02_Pin, J6 Conn_01x02_Pin, U2 DS18B20-air, U2 DS18B20-water, U4 TEMT6000, U4 Turbidity sensor, U5 GY-8511 UV sensor, U6 Water Level Sensor, U7 ESP32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

Commit message: PCB almost complete
Parts:
- U2: footprint Diplomna:DS18B20_3dmodel -> Diplomna:3pin_holes
Changed lines of the file:
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@@
       (effects (font (size 1.27 1.27)) (justify right))
     )
-    (property "Footprint" "Diplomna:DS18B20_3dmodel" (at 0 77.47 0)
+    (property "Footprint" "Diplomna:3pin_holes" (at 0 77.47 0)
       (effects (font (size 1.27 1.27)) hide)
     )
@@
       (effects (font (size 1.27 1.27)) (justify right))
     )
-    (property "Footprint" "Diplomna:DS18B20_3dmodel" (at 0 127 0)
-      (effects (font (size 1.27 1.27)) hide)
-    )
+    (property "Footprint" "Diplomna:3pin_holes" (at 0 127 0)
+      (effects (font (size 1.27 1.27)) hide)
+    )
